File: KiCad_Projects/ECE315_Lab6/ECE315_Lab6.sch (KiCad schematic (older format))
At the start: 0 parts

Commit message: Adding Temp Sensor, also annotated
Changed lines of the file:
@@
 $Descr A4 11693 8268
 encoding utf-8
-Sheet 1 5
+Sheet 1 6
 Title "Covid Temperature Sensor"
 Date "2020-11-29"
@@
 F1 "TouchSensor.sch" 50
 $EndSheet
+$Sheet
+S 4350 4850 2100 2550
+U 5FC8BA1D
+F0 "TempSensor.sch" 50
+F1 "TempSensor.sch" 50
+$EndSheet
+Text HLabel 6450 5200 0    50   Input ~ 0
+SDA
+Text HLabel 6450 5350 0    50   Input ~ 0
+SCL
 $EndSCHEMATC
