File: KiCad_Projects/ECE315_Lab6/MCU.sch (KiCad schematic (older format))
At the start: 15 parts, among them J301 Conn_01x05_Male, Q301 BC817-25-TP, U301 IC_CY8C4245PVI-482

Commit message: Adding Temp Sensor, also annotated
Parts:
- U301: symbol ECE315:IC_CY8C4245PVI-482 -> ECE315:IC_CY8C4245PVI-482-ECE315
Changed lines of the file:
@@
 $Descr A4 11693 8268
 encoding utf-8
-Sheet 4 5
+Sheet 4 6
 Title "MCU"
 Date "2020-09-24"
@@
 $EndComp
 $Comp
-L ECE315:IC_CY8C4245PVI-482 U301
+L ECE315:IC_CY8C4245PVI-482-ECE315 U301
 U 1 1 5F72B3A6
 P 7200 4300
+AR Path="/5F72B3A6" Ref="U301"  Part="1"
+AR Path="/5FC5B00F/5F72B3A6" Ref="U301"  Part="1"
 F 0 "U301" H 7500 7365 50  0000 C CNN
 F 1 "IC_CY8C4245PVI-482" H 7500 7274 50  0000 C CNN
