File: KiCad_Projects/ECE315_Lab6/PWR.sch (KiCad schematic (older format))
At the start: 7 parts

Commit message: Adding Temp Sensor, also annotated
Parts:
- gave numbers to parts that had none: 7
Changed lines of the file:
@@
 $Descr A4 11693 8268
 encoding utf-8
-Sheet 3 5
+Sheet 3 6
 Title ""
 Date ""
@@
 $EndDescr
 $Comp
-L dk_USB-DVI-HDMI-Connectors:10118193-0001LF J?
+L dk_USB-DVI-HDMI-Connectors:10118193-0001LF J302
 U 1 1 5F76702B
 P 2200 2950
-F 0 "J?" H 2264 3695 60  0000 C CNN
+F 0 "J302" H 2264 3695 60  0000 C CNN
 F 1 "10118193-0001LF" H 2264 3589 60  0000 C CNN
 F 2 "digikey-footprints:USB_Micro_B_Female_10118193-0001LF" H 2400 3150 60  0001 L CNN
@@
 $EndComp
 $Comp
-L ECE315:MCP2221A-I_SL U?
+L ECE315:MCP2221A-I_SL U303
 U 1 1 5F7685CC
 P 5150 2650
-F 0 "U?" H 5150 3517 50  0000 C CNN
+F 0 "U303" H 5150 3517 50  0000 C CNN
 F 1 "MCP2221A-I_SL" H 5150 3426 50  0000 C CNN
 F 2 "ECE315:SOIC127P600X175-14N" H 5150 2650 50  0001 L BNN
@@
 	4550 2950 2500 2950
 $Comp
-L power:GND #PWR?
+L power:GND #PWR0318
 U 1 1 5F76FCF2
 P 2800 3500
-F 0 "#PWR?" H 2800 3250 50  0001 C CNN
+F 0 "#PWR0318" H 2800 3250 50  0001 C CNN
 F 1 "GND" H 2805 3327 50  0000 C CNN
 F 2 "" H 2800 3500 50  0001 C CNN
@@
 	2800 3150 2800 3500
 $Comp
-L power:+5V #PWR?
+L power:+5V #PWR0320
 U 1 1 5F7704A1
 P 3050 2400
-F 0 "#PWR?" H 3050 2250 50  0001 C CNN
+F 0 "#PWR0320" H 3050 2250 50  0001 C CNN
 F 1 "+5V" H 3065 2573 50  0000 C CNN
 F 2 "" H 3050 2400 50  0001 C CNN
@@
 NoConn ~ 5750 2150
 $Comp
-L power:GND #PWR?
+L power:GND #PWR0324
 U 1 1 5F770E88
 P 6000 3400
-F 0 "#PWR?" H 6000 3150 50  0001 C CNN
+F 0 "#PWR0324" H 6000 3150 50  0001 C CNN
 F 1 "GND" H 6005 3227 50  0000 C CNN
 F 2 "" H 6000 3400 50  0001 C CNN
@@
 	6000 3250 6000 3400
 $Comp
-L Device:C C?
+L Device:C C305
 U 1 1 5F7715FA
 P 6850 2200
-F 0 "C?" H 6965 2246 50  0000 L CNN
+F 0 "C305" H 6965 2246 50  0000 L CNN
 F 1 "10uF" H 6965 2155 50  0000 L CNN
 F 2 "Capacitor_SMD:C_0805_2012Metric" H 6888 2050 50  0001 C CNN
@@
 	5750 2050 6850 2050
 $Comp
-L power:+3.3V #PWR?
+L power:+3.3V #PWR0325
 U 1 1 5F771E93
 P 6850 1650
-F 0 "#PWR?" H 6850 1500 50  0001 C CNN
+F 0 "#PWR0325" H 6850 1500 50  0001 C CNN
 F 1 "+3.3V" H 6865 1823 50  0000 C CNN
 F 2 "" H 6850 1650 50  0001 C CNN
@@
 $EndComp
 $Comp
-L power:+3.3V #PWR?
+L power:+3.3V #PWR0323
 U 1 1 5F77305A
 P 4250 1900
-F 0 "#PWR?" H 4250 1750 50  0001 C CNN
+F 0 "#PWR0323" H 4250 1750 50  0001 C CNN
 F 1 "+3.3V" H 4265 2073 50  0000 C CNN
 F 2 "" H 4250 1900 50  0001 C CNN
@@
 $EndComp
 $Comp
-L Device:R_US R?
+L Device:R_US R306
 U 1 1 5F77318F
 P 4250 2150
-F 0 "R?" H 4318 2196 50  0000 L CNN
+F 0 "R306" H 4318 2196 50  0000 L CNN
 F 1 "10K" H 4318 2105 50  0000 L CNN
 F 2 "Resistor_SMD:R_0805_2012Metric" V 4290 2140 50  0001 C CNN
@@
 Connection ~ 6850 2050
 $Comp
-L power:GND #PWR?
+L power:GND #PWR0326
 U 1 1 5F774389
 P 6850 2500
-F 0 "#PWR?" H 6850 2250 50  0001 C CNN
+F 0 "#PWR0326" H 6850 2250 50  0001 C CNN
 F 1 "GND" H 6855 2327 50  0000 C CNN
 F 2 "" H 6850 2500 50  0001 C CNN
@@
 	6400 2450 5750 2450
 $Comp
-L Regulator_Linear:TLV71333PDBV U?
+L Regulator_Linear:TLV71333PDBV U302
 U 1 1 5F775786
 P 2800 5350
-F 0 "U?" H 2800 5692 50  0000 C CNN
+F 0 "U302" H 2800 5692 50  0000 C CNN
 F 1 "TLV71333PDBV" H 2800 5601 50  0000 C CNN
 F 2 "Package_TO_SOT_SMD:SOT-23-5" H 2800 5675 50  0001 C CIN
@@
 $EndComp
 $Comp
-L power:+3.3V #PWR?
+L power:+3.3V #PWR0321
 U 1 1 5F7771CC
 P 3800 5000
-F 0 "#PWR?" H 3800 4850 50  0001 C CNN
+F 0 "#PWR0321" H 3800 4850 50  0001 C CNN
 F 1 "+3.3V" H 3815 5173 50  0000 C CNN
 F 2 "" H 3800 5000 50  0001 C CNN
@@
 $EndComp
 $Comp
-L power:+5V #PWR?
+L power:+5V #PWR0316
 U 1 1 5F777836
 P 1950 5150
-F 0 "#PWR?" H 1950 5000 50  0001 C CNN
+F 0 "#PWR0316" H 1950 5000 50  0001 C CNN
 F 1 "+5V" H 1965 5323 50  0000 C CNN
 F 2 "" H 1950 5150 50  0001 C CNN
@@
 $EndComp
 $Comp
-L power:GND #PWR?
+L power:GND #PWR0317
 U 1 1 5F778018
 P 1950 5900
-F 0 "#PWR?" H 1950 5650 50  0001 C CNN
+F 0 "#PWR0317" H 1950 5650 50  0001 C CNN
 F 1 "GND" H 1955 5727 50  0000 C CNN
 F 2 "" H 1950 5900 50  0001 C CNN
@@
 $EndComp
 $Comp
-L Device:C C?
+L Device:C C303
 U 1 1 5F778D7E
 P 1950 5600
-F 0 "C?" H 2065 5646 50  0000 L CNN
+F 0 "C303" H 2065 5646 50  0000 L CNN
 F 1 "10uF" H 2065 5555 50  0000 L CNN
 F 2 "Capacitor_SMD:C_0805_2012Metric" H 1988 5450 50  0001 C CNN
@@
 $EndComp
 $Comp
-L Device:C C?
+L Device:C C304
 U 1 1 5F77979B
 P 3800 5600
-F 0 "C?" H 3915 5646 50  0000 L CNN
+F 0 "C304" H 3915 5646 50  0000 L CNN
 F 1 "10uF" H 3915 5555 50  0000 L CNN
 F 2 "Capacitor_SMD:C_0805_2012Metric" H 3838 5450 50  0001 C CNN
@@
 $EndComp
 $Comp
-L power:GND #PWR?
+L power:GND #PWR0322
 U 1 1 5F779A45
 P 3800 5950
-F 0 "#PWR?" H 3800 5700 50  0001 C CNN
+F 0 "#PWR0322" H 3800 5700 50  0001 C CNN
 F 1 "GND" H 3805 5777 50  0000 C CNN
 F 2 "" H 3800 5950 50  0001 C CNN
@@
 Connection ~ 3800 5250
 $Comp
-L power:GND #PWR?
+L power:GND #PWR0319
 U 1 1 5F77C76F
 P 2800 5900
-F 0 "#PWR?" H 2800 5650 50  0001 C CNN
+F 0 "#PWR0319" H 2800 5650 50  0001 C CNN
 F 1 "GND" H 2805 5727 50  0000 C CNN
 F 2 "" H 2800 5900 50  0001 C CNN
