File: KiCad_Projects/ECE315_Lab6/TouchSensor.sch (KiCad schematic (older format))
At the start: 9 parts

Commit message: Added labels
Parts:
- removed JP?: SolderJumper_3_Open, symbol Jumper:SolderJumper_3_Open
- added SJ2: SolderJumper_3_Bridged12, symbol Jumper:SolderJumper_3_Bridged12
- SJ1: renamed from JP?; value SolderJumper_2_Open -> LED
- gave numbers to parts that had none: 1
Connections:
- net labels added: LEDA, Out
Changed lines of the file:
@@
 	4850 3850 5350 3850
 $Comp
-L dk_Rectangular-Connectors-Headers-Male-Pins:B4B-PH-K-S_LF__SN_ J?
+L dk_Rectangular-Connectors-Headers-Male-Pins:B4B-PH-K-S_LF__SN_ JP1
 U 1 1 5FC93282
 P 3350 1900
-F 0 "J?" V 3125 1908 50  0000 C CNN
+F 0 "JP1" V 3125 1908 50  0000 C CNN
 F 1 "B4B-PH-K-S_LF__SN_" V 3216 1908 50  0000 C CNN
 F 2 "digikey-footprints:PinHeader_1x4_P2mm_Drill1mm" H 3550 2100 60  0001 L CNN
@@
 Wire Wire Line
 	3550 2200 3550 2300
-$Comp
-L Jumper:SolderJumper_3_Open JP?
-U 1 1 5FC98BB9
-P 2200 3900
-F 0 "JP?" H 2200 4013 50  0000 C CNN
-F 1 "SolderJumper_3_Open" H 2200 4104 50  0000 C CNN
-F 2 "" H 2200 3900 50  0001 C CNN
-F 3 "~" H 2200 3900 50  0001 C CNN
-	1    2200 3900
-	-1   0    0    1
-$EndComp
 Wire Wire Line
 	4050 3650 2200 3650
 Wire Wire Line
 	2200 3650 2200 3750
-Wire Wire Line
-	2200 3750 2400 3750
-Wire Wire Line
-	2400 3750 2400 3900
-Connection ~ 2200 3750
 $Comp
 L power:+3.3V #PWR?
@@
 Wire Wire Line
 	2700 3900 2700 3850
-Connection ~ 2400 3900
 $Comp
 L power:GND #PWR?
@@
 	2350 5250 2900 5250
 $Comp
-L Jumper:SolderJumper_2_Open JP?
+L Jumper:SolderJumper_2_Open SJ1
 U 1 1 5FCA13F3
 P 1450 5250
-F 0 "JP?" H 1450 5455 50  0000 C CNN
-F 1 "SolderJumper_2_Open" H 1450 5364 50  0000 C CNN
+F 0 "SJ1" H 1450 5455 50  0000 C CNN
+F 1 "LED" H 1450 5364 50  0000 C CNN
 F 2 "" H 1450 5250 50  0001 C CNN
 F 3 "~" H 1450 5250 50  0001 C CNN
@@
 Wire Wire Line
 	2050 5250 1600 5250
+$Comp
+L Jumper:SolderJumper_3_Bridged12 SJ2
+U 1 1 5FC85CBF
+P 2200 3900
+F 0 "SJ2" H 2200 4013 50  0000 C CNN
+F 1 "SolderJumper_3_Bridged12" H 2200 4104 50  0000 C CNN
+F 2 "" H 2200 3900 50  0001 C CNN
+F 3 "~" H 2200 3900 50  0001 C CNN
+	1    2200 3900
+	-1   0    0    1
+$EndComp
+Text GLabel 1300 5250 0    50   Input ~ 0
+Out
+Text GLabel 2050 5250 0    50   Input ~ 0
+LEDA
+Text GLabel 3450 1900 2    50   Input ~ 0
+LEDA
+$Comp
+L power:+3.3V #PWR?
+U 1 1 5FC88D7B
+P 3950 2000
+F 0 "#PWR?" H 3950 1850 50  0001 C CNN
+F 1 "+3.3V" H 3965 2173 50  0000 C CNN
+F 2 "" H 3950 2000 50  0001 C CNN
+F 3 "" H 3950 2000 50  0001 C CNN
+	1    3950 2000
+	1    0    0    -1
+$EndComp
+Wire Wire Line
+	3450 2000 3950 2000
+Text GLabel 3650 2100 2    50   Input ~ 0
+Out
+Wire Wire Line
+	3450 2100 3650 2100
+Text GLabel 3900 3850 0    50   Input ~ 0
+Out
 $EndSCHEMATC

Commit message: Fixed labels
Changed lines of the file:
@@
 	-1   0    0    1
 $EndComp
-Text GLabel 1300 5250 0    50   Input ~ 0
-Out
-Text GLabel 2050 5250 0    50   Input ~ 0
-LEDA
-Text GLabel 3450 1900 2    50   Input ~ 0
-LEDA
 $Comp
 L power:+3.3V #PWR?
@@
 Wire Wire Line
 	3450 2000 3950 2000
-Text GLabel 3650 2100 2    50   Input ~ 0
-Out
 Wire Wire Line
 	3450 2100 3650 2100
-Text GLabel 3900 3850 0    50   Input ~ 0
+Text Label 3450 1900 0    50   ~ 0
+LEDA
+Text Label 1900 5250 0    50   ~ 0
+LEDA
+Wire Wire Line
+	1300 5250 1000 5250
+Text Label 1000 5250 0    50   ~ 0
+Out
+Text Label 3900 3850 0    50   ~ 0
+Out
+Text Label 3650 2100 0    50   ~ 0
 Out
 $EndSCHEMATC

Commit message: Adding Temp Sensor, also annotated
Parts:
- gave numbers to parts that had none: 1
Changed lines of the file:
@@
 $Descr A4 11693 8268
 encoding utf-8
-Sheet 5 5
+Sheet 5 6
 Title "Touch Sensor"
 Date "2020-12-02"
@@
 Connection ~ 5350 3300
 $Comp
-L power:+3.3V #PWR?
+L power:+3.3V #PWR0503
 U 1 1 5FC8EE54
 P 3250 3350
-F 0 "#PWR?" H 3250 3200 50  0001 C CNN
+F 0 "#PWR0503" H 3250 3200 50  0001 C CNN
 F 1 "+3.3V" H 3265 3523 50  0000 C CNN
 F 2 "" H 3250 3350 50  0001 C CNN
@@
 $EndComp
 $Comp
-L power:GND #PWR?
+L power:GND #PWR0504
 U 1 1 5FC93E7B
 P 3250 4400
-F 0 "#PWR?" H 3250 4150 50  0001 C CNN
+F 0 "#PWR0504" H 3250 4150 50  0001 C CNN
 F 1 "GND" H 3255 4227 50  0000 C CNN
 F 2 "" H 3250 4400 50  0001 C CNN
@@
 	4050 3850 3900 3850
 $Comp
-L Sensor_Touch:AT42QT1010-TSHR U?
+L Sensor_Touch:AT42QT1010-TSHR U501
 U 1 1 5FC95F40
 P 4450 3750
-F 0 "U?" H 4450 4231 50  0000 C CNN
+F 0 "U501" H 4450 4231 50  0000 C CNN
 F 1 "AT42QT1010-TSHR" H 4450 4140 50  0000 C CNN
 F 2 "Package_TO_SOT_SMD:SOT-23-6" H 4500 3500 50  0001 L CNN
@@
 $EndComp
 $Comp
-L power:GND #PWR?
+L power:GND #PWR0505
 U 1 1 5FC95128
 P 3550 2300
-F 0 "#PWR?" H 3550 2050 50  0001 C CNN
+F 0 "#PWR0505" H 3550 2050 50  0001 C CNN
 F 1 "GND" H 3555 2127 50  0000 C CNN
 F 2 "" H 3550 2300 50  0001 C CNN
@@
 	2200 3650 2200 3750
 $Comp
-L power:+3.3V #PWR?
+L power:+3.3V #PWR0502
 U 1 1 5FC9C33E
 P 2700 3850
-F 0 "#PWR?" H 2700 3700 50  0001 C CNN
+F 0 "#PWR0502" H 2700 3700 50  0001 C CNN
 F 1 "+3.3V" H 2715 4023 50  0000 C CNN
 F 2 "" H 2700 3850 50  0001 C CNN
@@
 	2700 3900 2700 3850
 $Comp
-L power:GND #PWR?
+L power:GND #PWR0501
 U 1 1 5FC9D19A
 P 1600 3900
-F 0 "#PWR?" H 1600 3650 50  0001 C CNN
+F 0 "#PWR0501" H 1600 3650 50  0001 C CNN
 F 1 "GND" H 1605 3727 50  0000 C CNN
 F 2 "" H 1600 3900 50  0001 C CNN
@@
 	2000 3900 1600 3900
 $Comp
-L power:GND #PWR?
+L power:GND #PWR0506
 U 1 1 5FC9DD85
 P 3750 5250
-F 0 "#PWR?" H 3750 5000 50  0001 C CNN
+F 0 "#PWR0506" H 3750 5000 50  0001 C CNN
 F 1 "GND" H 3755 5077 50  0000 C CNN
 F 2 "" H 3750 5250 50  0001 C CNN
@@
 $EndComp
 $Comp
-L power:+3.3V #PWR?
+L power:+3.3V #PWR0507
 U 1 1 5FC88D7B
 P 3950 2000
-F 0 "#PWR?" H 3950 1850 50  0001 C CNN
+F 0 "#PWR0507" H 3950 1850 50  0001 C CNN
 F 1 "+3.3V" H 3965 2173 50  0000 C CNN
 F 2 "" H 3950 2000 50  0001 C CNN
